Commit message: Add required xacro prefix to property tag and change arm_base_link to base_link

File: phantomx_arm_description/urdf/phantomx_macro.xacro (robot description, xacro)
@@ -1,13 +1,13 @@
 <?xml version="1.0" encoding="UTF-8"?>
 <robot xmlns:xacro="http://ros.org/wiki/xacro">
-   <property name="M_PI" value="3.14159"/>
-   <property name="M_SCALE" value="0.01"/>
+   <xacro:property name="M_PI" value="3.14159"/>
+   <xacro:property name="M_SCALE" value="0.01"/>
    <xacro:include filename="$(find phantomx_arm_description)/urdf/common_materials.xacro" />
    <xacro:include filename="$(find phantomx_arm_description)/urdf/robot_name_description.xacro" />
-   <!--link name="plate_top_link"/-->
-   <!--joint name="fixed" type="fixed">
+   <link name="plate_top_link"/>
+   <!--<joint name="fixed" type="fixed">
       <parent link="plate_top_link" />
       <child link="ph_base_link" />
-   </joint-->
+   </joint>-->
    <!-- REFERENCE: http://answers.gazebosim.org/question/4372/the-inertia-matrix-explained/ -->
    <xacro:macro name="phantomx_arm" params="prefix">
@@ -25,5 +25,5 @@
       </gazebo>
       <!-- links -->
-      <link name="arm_base_link">
+      <link name="base_link">
          <visual>
             <origin xyz="${M_SCALE*10} ${M_SCALE*10} ${M_SCALE*0}" rpy="${M_PI*0} ${M_PI*0} ${M_PI}" />
@@ -191,10 +191,10 @@
          <origin xyz="${M_SCALE*12.25} ${M_SCALE*0.2} ${M_SCALE*0.2}" rpy="${M_PI*0} ${M_PI*0} ${-M_PI/2}" />
          <parent link="plate_top_link" />
-         <child link="arm_base_link"/>
+         <child link="base_link"/>
          <axis xyz="0 1 0" />
       </joint>
       <joint name="joint_1" type="revolute">
          <origin xyz="${M_SCALE*0.125} ${M_SCALE*-3.25} ${M_SCALE*8.75}" rpy="${M_PI/2} ${M_PI*2} ${-M_PI/2}" />
-         <parent link="arm_base_link" />
+         <parent link="base_link" />
          <child link="link_1" />
          <axis xyz="0 1 0" />
